File: benchpsu_barreljack_adapter.kicad_sch (KiCad schematic)
At the start: 22 parts, among them J1 +, J2 -, J3 DC-044K-D020, SW1 SK22D15L5, U1 HT7525-1, U2 HT7525-1 (SOT89)

Commit message: Add files via upload
Parts:
- J1: Part Number 24.302.1 -> 24.302.1
- J2: Part Number 24.302.2 -> 24.302.2
- J3: Part Number DC-044K-D020 -> DC-044K-D020
- SW1: Part Number (none) -> SK22D15L5
- U1, U2: Part Number HT7525-1 -> HT7525-1
Changed lines of the file:
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@@
       (effects (font (size 1.27 1.27)) hide)
     )
-    (property "Part Number" " 24.302.2" (at 35.56 116.84 90)
+    (property "Part Number" "24.302.2" (at 35.56 116.84 90)
       (effects (font (size 1.27 1.27)) hide)
     )
@@
       (effects (font (size 1.27 1.27)) hide)
     )
-    (property "Part Number" " 24.302.1" (at 35.56 106.68 90)
+    (property "Part Number" "24.302.1" (at 35.56 106.68 90)
       (effects (font (size 1.27 1.27)) hide)
     )
@@
       (effects (font (size 1.27 1.27)) hide)
     )
-    (property "Part Number" " DC-044K-D020" (at 226.06 80.01 0)
+    (property "Part Number" "DC-044K-D020" (at 226.06 80.01 0)
       (effects (font (size 1.27 1.27)) hide)
     )
@@
       (effects (font (size 1.27 1.27)) hide)
     )
-    (property "Part Number" " HT7525-1" (at 133.35 86.233 0)
+    (property "Part Number" "HT7525-1" (at 133.35 86.233 0)
       (effects (font (size 1.27 1.27)) hide)
     )
@@
       (effects (font (size 1.27 1.27)) hide)
     )
-    (property "Part Number" " HT7525-1" (at 135.255 130.81 0)
+    (property "Part Number" "HT7525-1" (at 135.255 130.81 0)
       (effects (font (size 1.27 1.27)) hide)
     )
@@
       (effects (font (size 1.27 1.27)) hide)
     )
+    (property "Part Number" "SK22D15L5" (at 86.36 90.17 90)
+      (effects (font (size 1.27 1.27)) hide)
+    )
+    (property "Package" "" (at 86.36 90.17 90)
+      (effects (font (size 1.27 1.27)) hide)
+    )

Commit message: Updated project
Parts:
- C1, C2, C3, C4: Part Number (none) -> SM1061EMB072RB
- J1, J2: footprint benchpsu_barreljack_adapter:8x10pad -> benchpsu_barreljack_adapter:8x10pad_stitched
- R1, R2, R3, R4: value 100 -> 75; Part Number (none) -> FRC1206F75R0TS
Changed lines of the file:
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@@
       (effects (font (size 1.27 1.27)) (justify left))
     )
-    (property "Footprint" "benchpsu_barreljack_adapter:8x10pad" (at 35.56 116.84 0)
+    (property "Footprint" "benchpsu_barreljack_adapter:8x10pad_stitched" (at 35.56 116.84 0)
       (effects (font (size 1.27 1.27)) hide)
     )
@@
       (effects (font (size 1.27 1.27)) (justify left))
     )
-    (property "Footprint" "benchpsu_barreljack_adapter:8x10pad" (at 35.56 106.68 0)
+    (property "Footprint" "benchpsu_barreljack_adapter:8x10pad_stitched" (at 35.56 106.68 0)
       (effects (font (size 1.27 1.27)) hide)
     )
@@
       (effects (font (size 1.27 1.27)) hide)
     )
-    (property "Part Number" "" (at 142.875 140.208 0)
+    (property "Part Number" "SM1061EMB072RB" (at 142.875 140.208 0)
       (effects (font (size 1.27 1.27)) hide)
     )
@@
       (effects (font (size 1.27 1.27)))
     )
-    (property "Value" "100" (at 163.195 81.026 90)
+    (property "Value" "75" (at 163.195 81.026 90)
       (effects (font (size 1.27 1.27)))
     )
@@
       (effects (font (size 1.27 1.27)) hide)
     )
-    (property "Part Number" "" (at 163.195 83.693 90)
+    (property "Part Number" "FRC1206F75R0TS" (at 163.195 83.693 90)
       (effects (font (size 1.27 1.27)) hide)
     )
@@
       (effects (font (size 1.27 1.27)) hide)
     )
-    (property "Part Number" "" (at 127.635 140.208 0)
+    (property "Part Number" "SM1061EMB072RB" (at 127.635 140.208 0)
       (effects (font (size 1.27 1.27)) hide)
     )
@@
       (effects (font (size 1.27 1.27)) hide)
     )
-    (property "Part Number" "" (at 140.97 94.234 0)
+    (property "Part Number" "SM1061EMB072RB" (at 140.97 94.234 0)
       (effects (font (size 1.27 1.27)) hide)
     )
@@
       (effects (font (size 1.27 1.27)) hide)
     )
-    (property "Part Number" "" (at 125.73 94.234 0)
+    (property "Part Number" "SM1061EMB072RB" (at 125.73 94.234 0)
       (effects (font (size 1.27 1.27)) hide)
     )
@@
       (effects (font (size 1.27 1.27)))
     )
-    (property "Value" "100" (at 165.1 136.9314 90)
+    (property "Value" "75" (at 165.1 136.9314 90)
       (effects (font (size 1.27 1.27)))
     )
@@
       (effects (font (size 1.27 1.27)) hide)
     )
-    (property "Part Number" "" (at 165.1 132.08 90)
+    (property "Part Number" "FRC1206F75R0TS" (at 165.1 132.08 90)
       (effects (font (size 1.27 1.27)) hide)
     )
@@
       (effects (font (size 1.27 1.27)))
     )
-    (property "Value" "100" (at 163.195 93.6244 90)
+    (property "Value" "75" (at 163.195 93.6244 90)
       (effects (font (size 1.27 1.27)))
     )
@@
       (effects (font (size 1.27 1.27)) hide)
     )
-    (property "Part Number" "" (at 163.195 87.503 90)
+    (property "Part Number" "FRC1206F75R0TS" (at 163.195 87.503 90)
       (effects (font (size 1.27 1.27)) hide)
     )
@@
       (effects (font (size 1.27 1.27)))
     )
-    (property "Value" "100" (at 165.1 125.603 90)
+    (property "Value" "75" (at 165.1 125.603 90)
       (effects (font (size 1.27 1.27)))
     )
@@
       (effects (font (size 1.27 1.27)) hide)
     )
-    (property "Part Number" "" (at 165.1 128.27 90)
-      (effects (font (size 1.27 1.27)) hide)
-    )
+    (property "Part Number" "FRC1206F75R0TS" (at 165.1 128.27 90)
+      (effects (font (size 1.27 1.27)) hide)
+    )
